File: osshs-prog-module/osshs-prog-module.sch (KiCad schematic (older format))
At the start: 30 parts, among them J1 Conn_01x02, J2 Conn_02x03_Odd_Even, J3 Conn_01x04, J4 Conn_01x04, J5 USB_B_Mini, SW1 SW_Push, U1 MCP2551-I-SN, U2 FT232RL, U3 STM32F103RETx

Commit message: Fix annotations and footprints
Parts:
- gave numbers to parts that had none: 9
- renumbered U3 to U4
Changed lines of the file:
@@
 	5150 6650 5150 6550
 $Comp
-L power:+3.3V #PWR017
+L power:+3.3V #PWR018
 U 1 1 5E05712B
 P 5150 6550
-F 0 "#PWR017" H 5150 6400 50  0001 C CNN
+F 0 "#PWR018" H 5150 6400 50  0001 C CNN
 F 1 "+3.3V" H 5165 6723 50  0000 C CNN
 F 2 "" H 5150 6550 50  0001 C CNN
@@
 	5150 7350 5150 7250
 $Comp
-L power:+3.3V #PWR018
+L power:+3.3V #PWR019
 U 1 1 5E070341
 P 5150 7250
-F 0 "#PWR018" H 5150 7100 50  0001 C CNN
+F 0 "#PWR019" H 5150 7100 50  0001 C CNN
 F 1 "+3.3V" H 5165 7423 50  0000 C CNN
 F 2 "" H 5150 7250 50  0001 C CNN
@@
 	6050 7350 6050 7450
 $Comp
-L power:GND #PWR021
+L power:GND #PWR024
 U 1 1 5E099AA7
 P 6050 7450
-F 0 "#PWR021" H 6050 7200 50  0001 C CNN
+F 0 "#PWR024" H 6050 7200 50  0001 C CNN
 F 1 "GND" H 6055 7277 50  0000 C CNN
 F 2 "" H 6050 7450 50  0001 C CNN
@@
 $EndComp
 $Comp
-L power:GND #PWR019
+L power:GND #PWR020
 U 1 1 5E4F451A
 P 5200 5550
-F 0 "#PWR019" H 5200 5300 50  0001 C CNN
+F 0 "#PWR020" H 5200 5300 50  0001 C CNN
 F 1 "GND" H 5205 5377 50  0000 C CNN
 F 2 "" H 5200 5550 50  0001 C CNN
@@
 $EndComp
 $Comp
-L power:+5V #PWR020
+L power:+5V #PWR023
 U 1 1 5E4FEAA8
 P 5650 4750
-F 0 "#PWR020" H 5650 4600 50  0001 C CNN
+F 0 "#PWR023" H 5650 4600 50  0001 C CNN
 F 1 "+5V" H 5665 4923 50  0000 C CNN
 F 2 "" H 5650 4750 50  0001 C CNN
@@
 Text GLabel 1450 2700 0    50   Input ~ 0
 USART2_RESET
-$Comp
-L Regulator_Linear:MCP1700-3302E_SOT23 U?
-U 1 1 5E57B632
-P 5250 3200
-F 0 "U?" H 5250 3442 50  0000 C CNN
-F 1 "MCP1700-3302E_SOT23" H 5250 3351 50  0000 C CNN
-F 2 "Package_TO_SOT_SMD:SOT-23" H 5250 3425 50  0001 C CNN
-F 3 "http://ww1.microchip.com/downloads/en/DeviceDoc/20001826D.pdf" H 5250 3200 50  0001 C CNN
-	1    5250 3200
-	1    0    0    -1
-$EndComp
-Wire Wire Line
-	5250 3500 5250 3600
-$Comp
-L power:GND #PWR?
-U 1 1 5E59C063
-P 5250 3600
-F 0 "#PWR?" H 5250 3350 50  0001 C CNN
-F 1 "GND" H 5255 3427 50  0000 C CNN
-F 2 "" H 5250 3600 50  0001 C CNN
-F 3 "" H 5250 3600 50  0001 C CNN
-	1    5250 3600
-	1    0    0    -1
-$EndComp
-Wire Wire Line
-	4950 3200 4850 3200
-Wire Wire Line
-	4850 3200 4850 3100
-Wire Wire Line
-	5550 3200 5650 3200
-Wire Wire Line
-	5650 3200 5650 3100
-$Comp
-L power:+5V #PWR?
-U 1 1 5E5B2704
-P 4850 3100
-F 0 "#PWR?" H 4850 2950 50  0001 C CNN
-F 1 "+5V" H 4865 3273 50  0000 C CNN
-F 2 "" H 4850 3100 50  0001 C CNN
-F 3 "" H 4850 3100 50  0001 C CNN
-	1    4850 3100
-	1    0    0    -1
-$EndComp
-$Comp
-L power:+3.3V #PWR?
-U 1 1 5E5CEFD9
-P 5650 3100
-F 0 "#PWR?" H 5650 2950 50  0001 C CNN
-F 1 "+3.3V" H 5665 3273 50  0000 C CNN
-F 2 "" H 5650 3100 50  0001 C CNN
-F 3 "" H 5650 3100 50  0001 C CNN
-	1    5650 3100
-	1    0    0    -1
-$EndComp
 Wire Wire Line
 	6800 1350 6800 1450
@@
 	6800 950  6800 850
 $Comp
-L power:GND #PWR?
+L power:GND #PWR026
 U 1 1 5E5DEB72
 P 6800 1450
-F 0 "#PWR?" H 6800 1200 50  0001 C CNN
+F 0 "#PWR026" H 6800 1200 50  0001 C CNN
 F 1 "GND" H 6805 1277 50  0000 C CNN
 F 2 "" H 6800 1450 50  0001 C CNN
@@
 $EndComp
 $Comp
-L Device:C C?
+L Device:C C4
 U 1 1 5E5DEB7E
 P 6800 1100
-F 0 "C?" H 6685 1054 50  0000 R CNN
+F 0 "C4" H 6685 1054 50  0000 R CNN
 F 1 "100nF" H 6685 1145 50  0000 R CNN
 F 2 "Capacitor_SMD:C_0805_2012Metric" H 6838 950 50  0001 C CNN
@@
 $EndComp
 $Comp
-L power:+3.3V #PWR?
+L power:+3.3V #PWR025
 U 1 1 5E5F87F5
 P 6800 750
-F 0 "#PWR?" H 6800 600 50  0001 C CNN
+F 0 "#PWR025" H 6800 600 50  0001 C CNN
 F 1 "+3.3V" H 6815 923 50  0000 C CNN
 F 2 "" H 6800 750 50  0001 C CNN
@@
 SWDIO
 $Comp
-L power:GND #PWR022
+L power:GND #PWR029
 U 1 1 5DEBBFB0
 P 9650 6100
-F 0 "#PWR022" H 9650 5850 50  0001 C CNN
+F 0 "#PWR029" H 9650 5850 50  0001 C CNN
 F 1 "GND" H 9655 5927 50  0000 C CNN
 F 2 "" H 9650 6100 50  0001 C CNN
@@
 	9250 6000 9350 6000
 $Comp
-L power:+3.3V #PWR023
+L power:+3.3V #PWR030
 U 1 1 5DEAFF7F
 P 9750 2000
-F 0 "#PWR023" H 9750 1850 50  0001 C CNN
+F 0 "#PWR030" H 9750 1850 50  0001 C CNN
 F 1 "+3.3V" H 9765 2173 50  0000 C CNN
 F 2 "" H 9750 2000 50  0001 C CNN
@@
 	8750 2450 8600 2450
 $Comp
-L MCU_ST_STM32F1:STM32F103RETx U3
+L MCU_ST_STM32F1:STM32F103RETx U4
 U 1 1 5DE66C62
 P 9450 4050
-F 0 "U3" H 9450 2161 50  0000 C CNN
+F 0 "U4" H 9450 2161 50  0000 C CNN
 F 1 "STM32F103RETx" H 9450 2070 50  0000 C CNN
 F 2 "Package_QFP:LQFP-64_10x10mm_P0.5mm" H 8850 2350 50  0001 R CNN
@@
 $EndComp
 $Comp
-L Device:C C?
+L Device:C C5
 U 1 1 5E663F55
 P 7200 1100
-F 0 "C?" H 7085 1054 50  0000 R CNN
+F 0 "C5" H 7085 1054 50  0000 R CNN
 F 1 "100nF" H 7085 1145 50  0000 R CNN
 F 2 "Capacitor_SMD:C_0805_2012Metric" H 7238 950 50  0001 C CNN
@@
 $EndComp
 $Comp
-L Device:C C?
+L Device:C C6
 U 1 1 5E669B40
 P 7600 1100
-F 0 "C?" H 7485 1054 50  0000 R CNN
+F 0 "C6" H 7485 1054 50  0000 R CNN
 F 1 "100nF" H 7485 1145 50  0000 R CNN
 F 2 "Capacitor_SMD:C_0805_2012Metric" H 7638 950 50  0001 C CNN
@@
 $EndComp
 $Comp
-L Device:C C?
+L Device:C C7
 U 1 1 5E66F58C
 P 8000 1100
-F 0 "C?" H 7885 1054 50  0000 R CNN
+F 0 "C7" H 7885 1054 50  0000 R CNN
 F 1 "100nF" H 7885 1145 50  0000 R CNN
 F 2 "Capacitor_SMD:C_0805_2012Metric" H 8038 950 50  0001 C CNN
@@
 $EndComp
 $Comp
-L Device:C C?
+L Device:C C8
 U 1 1 5E67AA19
 P 8400 1100
-F 0 "C?" H 8285 1054 50  0000 R CNN
+F 0 "C8" H 8285 1054 50  0000 R CNN
 F 1 "100nF" H 8285 1145 50  0000 R CNN
 F 2 "Capacitor_SMD:C_0805_2012Metric" H 8438 950 50  0001 C CNN
@@
 $EndComp
 $Comp
-L Device:C C?
+L Device:C C9
 U 1 1 5E686270
 P 8800 1100
-F 0 "C?" H 8685 1054 50  0000 R CNN
+F 0 "C9" H 8685 1054 50  0000 R CNN
 F 1 "10uF" H 8685 1145 50  0000 R CNN
 F 2 "Capacitor_SMD:C_0805_2012Metric" H 8838 950 50  0001 C CNN
@@
 	9350 950  9350 850
 $Comp
-L power:GND #PWR?
+L power:GND #PWR028
 U 1 1 5E6CD83A
 P 9350 1450
-F 0 "#PWR?" H 9350 1200 50  0001 C CNN
+F 0 "#PWR028" H 9350 1200 50  0001 C CNN
 F 1 "GND" H 9355 1277 50  0000 C CNN
 F 2 "" H 9350 1450 50  0001 C CNN
@@
 $EndComp
 $Comp
-L Device:C C?
+L Device:C C10
 U 1 1 5E6CD840
 P 9350 1100
-F 0 "C?" H 9235 1054 50  0000 R CNN
+F 0 "C10" H 9235 1054 50  0000 R CNN
 F 1 "100nF" H 9235 1145 50  0000 R CNN
 F 2 "Capacitor_SMD:C_0805_2012Metric" H 9388 950 50  0001 C CNN
@@
 $EndComp
 $Comp
-L power:+3.3V #PWR?
+L power:+3.3V #PWR027
 U 1 1 5E6CD846
 P 9350 750
-F 0 "#PWR?" H 9350 600 50  0001 C CNN
+F 0 "#PWR027" H 9350 600 50  0001 C CNN
 F 1 "+3.3V" H 9365 923 50  0000 C CNN
 F 2 "" H 9350 750 50  0001 C CNN
@@
 	9350 1350 9750 1350
 $Comp
-L Device:C C?
+L power:+3.3V #PWR022
+U 1 1 5E5CEFD9
+P 5650 3100
+F 0 "#PWR022" H 5650 2950 50  0001 C CNN
+F 1 "+3.3V" H 5665 3273 50  0000 C CNN
+F 2 "" H 5650 3100 50  0001 C CNN
+F 3 "" H 5650 3100 50  0001 C CNN
+	1    5650 3100
+	1    0    0    -1
+$EndComp
+$Comp
+L power:+5V #PWR017
+U 1 1 5E5B2704
+P 4850 3100
+F 0 "#PWR017" H 4850 2950 50  0001 C CNN
+F 1 "+5V" H 4865 3273 50  0000 C CNN
+F 2 "" H 4850 3100 50  0001 C CNN
+F 3 "" H 4850 3100 50  0001 C CNN
+	1    4850 3100
+	1    0    0    -1
+$EndComp
+Wire Wire Line
+	5650 3200 5650 3100
+Wire Wire Line
+	5550 3200 5650 3200
+Wire Wire Line
+	4850 3200 4850 3100
+Wire Wire Line
+	4950 3200 4850 3200
+$Comp
+L power:GND #PWR021
+U 1 1 5E59C063
+P 5250 3600
+F 0 "#PWR021" H 5250 3350 50  0001 C CNN
+F 1 "GND" H 5255 3427 50  0000 C CNN
+F 2 "" H 5250 3600 50  0001 C CNN
+F 3 "" H 5250 3600 50  0001 C CNN
+	1    5250 3600
+	1    0    0    -1
+$EndComp
+Wire Wire Line
+	5250 3500 5250 3600
+$Comp
+L Regulator_Linear:MCP1700-3302E_SOT23 U3
+U 1 1 5E57B632
+P 5250 3200
+F 0 "U3" H 5250 3442 50  0000 C CNN
+F 1 "MCP1700-3302E_SOT23" H 5250 3351 50  0000 C CNN
+F 2 "Package_TO_SOT_SMD:SOT-23" H 5250 3425 50  0001 C CNN
+F 3 "http://ww1.microchip.com/downloads/en/DeviceDoc/20001826D.pdf" H 5250 3200 50  0001 C CNN
+	1    5250 3200
+	1    0    0    -1
+$EndComp
+$Comp
+L Device:C C11
 U 1 1 5E6CD850
 P 9750 1100
-F 0 "C?" H 9635 1054 50  0000 R CNN
+F 0 "C11" H 9635 1054 50  0000 R CNN
 F 1 "1uF" H 9635 1145 50  0000 R CNN
 F 2 "Capacitor_SMD:C_0805_2012Metric" H 9788 950 50  0001 C CNN
